File: DDS.sch (KiCad schematic (older format))
At the start: 169 parts, among them J1 Conn_01x05_Male, J2 USB_B_Mini, J3 Barrel_Jack_Switch, J4 Conn_Coaxial, J5 Conn_Coaxial, J6 Conn_Coaxial, U1 5M160ZT100, U2 LM317_SOT-223, U3 MCP2210x-SS, U4 ETXO-H33CL-100.000, U5 IS61LF12836, U6 DAC5687IPZP, Y1 12Meg

Commit message: new changes
Parts:
- removed R14: 22, Resistor_SMD:R_0603_1608Metric, symbol Device:R_Small
- removed R16: 1k, Resistor_SMD:R_0603_1608Metric, symbol Device:R_Small
- removed R3: 510, Resistor_SMD:R_0603_1608Metric, symbol Device:R_Small
- removed R4: 220, Resistor_SMD:R_0603_1608Metric, symbol Device:R_Small
- removed TP10, TP11, TP12, TP13, TP14, TP15, TP16, TP17, TP18, TP19, TP20, TP21, TP22, TP23, TP24, TP25, TP26, TP27, TP28, TP29, TP3, TP30, TP31, TP32, TP33, TP34, TP37, TP38, TP39, TP4, TP40, TP41, TP42, TP43, TP46, TP47, TP48, TP49, TP50, TP51, TP52, TP53, TP54, TP55, TP56, TP57, TP58, TP59, TP6, TP60, TP61, TP62, TP63, TP64, TP65, TP66, TP67, TP68, TP69, TP7, TP70, TP71, TP72, TP73, TP74, TP75, TP76, TP77, TP78, TP79, TP8, TP80, TP81: TestPoint, TestPoint:TestPoint_Pad_D1.0mm, symbol Connector:TestPoint
- removed U2: LM317_SOT-223, Package_TO_SOT_SMD:SOT-223-3_TabPin2, symbol Regulator_Linear:LM317_SOT-223
- added C26: 1u, Capacitor_SMD:C_0603_1608Metric, symbol Device:C_Small
- added H1, H2, H3, H4: MountingHole, MountingHole:MountingHole_3.2mm_M3, symbol Mechanical:MountingHole
- added J7: Debug_Header, Connector_PinHeader_2.54mm:PinHeader_1x09_P2.54mm_Vertical, symbol Connector:Conn_01x09_Male
- added R22: 1k, Resistor_SMD:R_0603_1608Metric, symbol Device:R_Small
- added RN3, RN4, RN5, RN6: R_Pack08, HS2_parts:CAY16-470J8LF, symbol Device:R_Pack08
- added U2: AZ1117-1.8, Package_TO_SOT_SMD:SOT-223-3_TabPin2, symbol Regulator_Linear:AZ1117-1.8
- J1: footprint Connector_PinHeader_1.27mm:PinHeader_1x05_P1.27mm_Vertical -> Connector_PinHeader_2.54mm:PinHeader_1x05_P2.54mm_Vertical
- R2: value 22 -> 100
- gave numbers to parts that had none: 1
Connections:
- net labels added: SRAM_CLK, TCK, TDI, TDO, TMS
- net labels removed: HS_CLK_EN, LS_CLK, MODE, ZZ, ~ADSP, ~ADV, ~BWE
- wire segments 544 -> 520
- no-connect marks 9 -> 7
Other:
- note removed: "Optional Termination - Omitted \n(we'll see if I regret this later)"
- moved on the sheet: C1, C10, C11, C12, C13, C14, C15, C16, C17, C18, C19, C2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
